Commit message: plugins naming fixed startup sequence for unitree_cmd_vel disabled

File: src/g1_description/urdf/g1_29dof.urdf (robot description, URDF)
Before this commit: robot g1_29dof, 40 links, 39 joints
Links:
- removed link mid360_link
- added link utlidar_lidar
Joints:
- joint mid360_joint: child mid360_link -> utlidar_lidar
